File: pcb/esp8266-module.sch (KiCad schematic (older format))
At the start: 15 parts, among them U1 ESP-12E

Commit message: re-map I/O
Parts:
- added C-SWITCH1: C, Capacitor_SMD:C_0805_2012Metric, symbol Device:C
- added R-SWITCH1: 10K, Resistor_SMD:R_0805_2012Metric, symbol Device:R
- added SW-SWITCH1: SW_Push, Button_Switch_SMD:SW_SPST_B3U-1000P-B, symbol Switch:SW_Push
Connections:
- net GND: now also C-SWITCH1.2, SW-SWITCH1.2
- net VDD: now also R-SWITCH1.2
- net GPIO_14: now reaches U1.5 (GPIO14)
- net GPIO_14: now also C-SWITCH1.1, R-SWITCH1.1, SW-SWITCH1.1
Other:
- moved on the sheet: C-PIR1, J-PIR1, R-PIR1
Changed lines of the file:
@@
 EESchema Schematic File Version 4
+LIBS:esp8266-module-cache
 EELAYER 26 0
 EELAYER END
@@
 L Connector:Conn_01x03_Male J-PIR1
 U 1 1 5DB3E48F
-P 3500 3500
-F 0 "J-PIR1" H 3606 3778 50  0000 C CNN
-F 1 "Conn_01x03_Male" H 3606 3687 50  0000 C CNN
-F 2 "solder_pads:solderpads_1x3" H 3500 3500 50  0001 C CNN
-F 3 "~" H 3500 3500 50  0001 C CNN
-	1    3500 3500
+P 4350 3150
+F 0 "J-PIR1" H 4456 3428 50  0000 C CNN
+F 1 "Conn_01x03_Male" H 4456 3337 50  0000 C CNN
+F 2 "solder_pads:solderpads_1x3" H 4350 3150 50  0001 C CNN
+F 3 "~" H 4350 3150 50  0001 C CNN
+	1    4350 3150
 	1    0    0    -1
 $EndComp
@@
 L power:VDD #PWR0105
 U 1 1 5DB3E9A6
-P 3800 3400
-F 0 "#PWR0105" H 3800 3250 50  0001 C CNN
-F 1 "VDD" H 3817 3573 50  0000 C CNN
-F 2 "" H 3800 3400 50  0001 C CNN
-F 3 "" H 3800 3400 50  0001 C CNN
-	1    3800 3400
-	1    0    0    -1
-$EndComp
-Wire Wire Line
-	3800 3400 3700 3400
-Wire Wire Line
-	3800 3600 3700 3600
-Wire Wire Line
-	3700 3500 4000 3500
+P 4650 3050
+F 0 "#PWR0105" H 4650 2900 50  0001 C CNN
+F 1 "VDD" H 4667 3223 50  0000 C CNN
+F 2 "" H 4650 3050 50  0001 C CNN
+F 3 "" H 4650 3050 50  0001 C CNN
+	1    4650 3050
+	1    0    0    -1
+$EndComp
+Wire Wire Line
+	4650 3050 4550 3050
+Wire Wire Line
+	4650 3250 4550 3250
+Wire Wire Line
+	4550 3150 4850 3150
 $Comp
 L Device:R R-PIR1
 U 1 1 5DB40212
-P 4000 3300
-F 0 "R-PIR1" H 4070 3346 50  0000 L CNN
-F 1 "10K" H 4070 3255 50  0000 L CNN
-F 2 "Resistor_SMD:R_0805_2012Metric" V 3930 3300 50  0001 C CNN
-F 3 "~" H 4000 3300 50  0001 C CNN
-	1    4000 3300
+P 4850 2950
+F 0 "R-PIR1" H 4920 2996 50  0000 L CNN
+F 1 "10K" H 4920 2905 50  0000 L CNN
+F 2 "Resistor_SMD:R_0805_2012Metric" V 4780 2950 50  0001 C CNN
+F 3 "~" H 4850 2950 50  0001 C CNN
+	1    4850 2950
 	1    0    0    -1
 $EndComp
@@
 L power:VDD #PWR0107
 U 1 1 5DB40338
-P 4000 3100
-F 0 "#PWR0107" H 4000 2950 50  0001 C CNN
-F 1 "VDD" H 4017 3273 50  0000 C CNN
-F 2 "" H 4000 3100 50  0001 C CNN
-F 3 "" H 4000 3100 50  0001 C CNN
-	1    4000 3100
-	1    0    0    -1
-$EndComp
-Wire Wire Line
-	4000 3100 4000 3150
-Wire Wire Line
-	4000 3450 4000 3500
-Connection ~ 4000 3500
-Wire Wire Line
-	4000 3500 4250 3500
-Text Label 4250 3500 0    50   ~ 0
+P 4850 2750
+F 0 "#PWR0107" H 4850 2600 50  0001 C CNN
+F 1 "VDD" H 4867 2923 50  0000 C CNN
+F 2 "" H 4850 2750 50  0001 C CNN
+F 3 "" H 4850 2750 50  0001 C CNN
+	1    4850 2750
+	1    0    0    -1
+$EndComp
+Wire Wire Line
+	4850 2750 4850 2800
+Wire Wire Line
+	4850 3100 4850 3150
+Connection ~ 4850 3150
+Wire Wire Line
+	4850 3150 5100 3150
+Text Label 5100 3150 0    50   ~ 0
 GPIO_13
 $Comp
 L Device:C C-PIR1
 U 1 1 5DB4523C
-P 4000 3650
-F 0 "C-PIR1" H 4115 3696 50  0000 L CNN
-F 1 "C" H 4115 3605 50  0000 L CNN
-F 2 "Capacitor_SMD:C_0805_2012Metric" H 4038 3500 50  0001 C CNN
-F 3 "~" H 4000 3650 50  0001 C CNN
-	1    4000 3650
+P 4850 3300
+F 0 "C-PIR1" H 4965 3346 50  0000 L CNN
+F 1 "C" H 4965 3255 50  0000 L CNN
+F 2 "Capacitor_SMD:C_0805_2012Metric" H 4888 3150 50  0001 C CNN
+F 3 "~" H 4850 3300 50  0001 C CNN
+	1    4850 3300
 	1    0    0    -1
 $EndComp
@@
 L power:GND #PWR0103
 U 1 1 5DB474CB
-P 3900 3800
-F 0 "#PWR0103" H 3900 3550 50  0001 C CNN
-F 1 "GND" H 3905 3627 50  0000 C CNN
-F 2 "" H 3900 3800 50  0001 C CNN
-F 3 "" H 3900 3800 50  0001 C CNN
-	1    3900 3800
+P 4750 3450
+F 0 "#PWR0103" H 4750 3200 50  0001 C CNN
+F 1 "GND" H 4755 3277 50  0000 C CNN
+F 2 "" H 4750 3450 50  0001 C CNN
+F 3 "" H 4750 3450 50  0001 C CNN
+	1    4750 3450
 	1    0    0    -1
 $EndComp
@@
 Connection ~ 1100 2850
 Wire Wire Line
-	4000 3800 3900 3800
-Wire Wire Line
-	3800 3600 3800 3800
-Wire Wire Line
-	3800 3800 3900 3800
-Connection ~ 3900 3800
+	4850 3450 4750 3450
+Wire Wire Line
+	4650 3250 4650 3450
+Wire Wire Line
+	4650 3450 4750 3450
+Connection ~ 4750 3450
+$Comp
+L Device:R R-SWITCH1
+U 1 1 5DB36EB9
+P 2200 1900
+F 0 "R-SWITCH1" V 1993 1900 50  0000 C CNN
+F 1 "10K" V 2084 1900 50  0000 C CNN
+F 2 "Resistor_SMD:R_0805_2012Metric" V 2130 1900 50  0001 C CNN
+F 3 "~" H 2200 1900 50  0001 C CNN
+	1    2200 1900
+	0    1    1    0
+$EndComp
+Wire Wire Line
+	2750 1900 2350 1900
+Wire Wire Line
+	2050 1900 2000 1900
+Wire Wire Line
+	2000 1900 2000 1700
+Connection ~ 2000 1700
+Text Label 2500 1900 0    50   ~ 0
+GPIO_14
+$Comp
+L Switch:SW_Push SW-SWITCH1
+U 1 1 5DB3958C
+P 3500 3250
+F 0 "SW-SWITCH1" H 3500 3535 50  0000 C CNN
+F 1 "SW_Push" H 3500 3444 50  0000 C CNN
+F 2 "Button_Switch_SMD:SW_SPST_B3U-1000P-B" H 3500 3450 50  0001 C CNN
+F 3 "" H 3500 3450 50  0001 C CNN
+	1    3500 3250
+	1    0    0    -1
+$EndComp
+$Comp
+L power:GND #PWR0108
+U 1 1 5DB39593
+P 3700 3350
+F 0 "#PWR0108" H 3700 3100 50  0001 C CNN
+F 1 "GND" H 3705 3177 50  0000 C CNN
+F 2 "" H 3700 3350 50  0001 C CNN
+F 3 "" H 3700 3350 50  0001 C CNN
+	1    3700 3350
+	1    0    0    -1
+$EndComp
+Wire Wire Line
+	3300 3250 3200 3250
+Wire Wire Line
+	3700 3250 3700 3350
+Text Label 3100 3250 0    50   ~ 0
+GPIO_14
+$Comp
+L Device:C C-SWITCH1
+U 1 1 5DB3959C
+P 3200 3450
+F 0 "C-SWITCH1" H 3315 3496 50  0000 L CNN
+F 1 "C" H 3315 3405 50  0000 L CNN
+F 2 "Capacitor_SMD:C_0805_2012Metric" H 3238 3300 50  0001 C CNN
+F 3 "~" H 3200 3450 50  0001 C CNN
+	1    3200 3450
+	1    0    0    -1
+$EndComp
+$Comp
+L power:GND #PWR0109
+U 1 1 5DB395A3
+P 3200 3700
+F 0 "#PWR0109" H 3200 3450 50  0001 C CNN
+F 1 "GND" H 3205 3527 50  0000 C CNN
+F 2 "" H 3200 3700 50  0001 C CNN
+F 3 "" H 3200 3700 50  0001 C CNN
+	1    3200 3700
+	1    0    0    -1
+$EndComp
+Wire Wire Line
+	3200 3600 3200 3700
+Wire Wire Line
+	3200 3300 3200 3250
+Connection ~ 3200 3250
+Wire Wire Line
+	3200 3250 3100 3250
 $EndSCHEMATC
